File: KiCad/6N6P_hybrid.kicad_pcb (KiCad board)
At the start: 2 copper layers, 165.1 x 62.9 mm, 45 parts, among them J1 Screw_Terminal_01x02, J2 Screw_Terminal_01x02, J3 Screw_Terminal_01x02, J4 Screw_Terminal_01x02, J5 Screw_Terminal_01x03, J6 Screw_Terminal_01x03, J7 Screw_Terminal_01x02, J8 Screw_Terminal_01x03, J9 Screw_Terminal_01x01, Q1 BC107, U1 LTC1151CN8, U2 LTC1151CN8

Commit message: Add files via upload
Parts:
- added C10: 100uF/400V, Capacitor_THT:CP_Radial_D25.0mm_P10.00mm_SnapIn, F.Cu at (62.9, 121.9)
- added C11: 4700uF/35V, Capacitor_THT:CP_Radial_D12.5mm_P7.50mm, F.Cu at (75.6, 151.4)
- added C13: 4700uF/35V, Capacitor_THT:CP_Radial_D12.5mm_P7.50mm, F.Cu at (61.6, 158.6)
- added C14: C, Capacitor_THT:C_Disc_D8.0mm_W5.0mm_P10.00mm, F.Cu at (98.3, 131.4)
- added C15: C, Capacitor_THT:C_Disc_D8.0mm_W5.0mm_P10.00mm, F.Cu at (50.8, 150.5)
- added C16: C, Capacitor_THT:C_Disc_D8.0mm_W5.0mm_P10.00mm, F.Cu at (84.5, 149.1)
- added D10: 1N4001, Diode_THT:D_DO-41_SOD81_P10.16mm_Horizontal, F.Cu at (34.3, 154.9)
- added D3: 1N4001, Diode_THT:D_DO-41_SOD81_P10.16mm_Horizontal, F.Cu at (43.2, 123.8)
- added D4: 1N4001, Diode_THT:D_DO-41_SOD81_P10.16mm_Horizontal, F.Cu at (43.2, 130.2)
- added D5: 1N4001, Diode_THT:D_DO-41_SOD81_P10.16mm_Horizontal, F.Cu at (33.0, 118.1)
- added D6: 1N4001, Diode_THT:D_DO-41_SOD81_P10.16mm_Horizontal, F.Cu at (34.3, 112.4)
- added D7: 1N4001, Diode_THT:D_DO-41_SOD81_P10.16mm_Horizontal, F.Cu at (43.2, 143.5)
- added D8: 1N4001, Diode_THT:D_DO-41_SOD81_P10.16mm_Horizontal, F.Cu at (43.2, 137.8)
- added D9: 1N4001, Diode_THT:D_DO-41_SOD81_P10.16mm_Horizontal, F.Cu at (33.0, 149.2)
- added F1: Fuse, Fuse:Fuseholder_Clip-5x20mm_Keystone_3517_Inline_P23.11x6.76mm_D1.70mm_Horizontal, F.Cu at (73.2, 134.6)
- added F2: Fuse, Fuse:Fuseholder_Clip-5x20mm_Keystone_3517_Inline_P23.11x6.76mm_D1.70mm_Horizontal, F.Cu at (73.2, 143.5)
- added J10: Screw_Terminal_01x03, Connector_Phoenix_MSTB:PhoenixContact_MSTBA_2,5_3-G-5,08_1x03_P5.08mm_Horizontal, F.Cu at (90.8, 149.2)
- added J11: Screw_Terminal_01x01, Connector_Pin:Pin_D1.1mm_L8.5mm_W2.5mm_FlatFork, F.Cu at (26.7, 118.1)
- added J12: Screw_Terminal_01x01, Connector_Pin:Pin_D1.1mm_L8.5mm_W2.5mm_FlatFork, F.Cu at (26.7, 130.2)
- added J13: Screw_Terminal_01x01, Connector_Pin:Pin_D1.1mm_L8.5mm_W2.5mm_FlatFork, F.Cu at (26.7, 149.2)
- added J14: Screw_Terminal_01x01, Connector_Pin:Pin_D1.1mm_L8.5mm_W2.5mm_FlatFork, F.Cu at (26.7, 137.8)
- added J15: PSU ground, Connector_Pin:Pin_D1.1mm_L8.5mm_W2.5mm_FlatFork, F.Cu at (92.1, 114.9)
- added J16: Screw_Terminal_01x01, Connector_Pin:Pin_D1.1mm_L8.5mm_W2.5mm_FlatFork, F.Cu at (92.1, 124.5)
- added J17: center tap, Connector_Pin:Pin_D1.1mm_L8.5mm_W2.5mm_FlatFork, F.Cu at (40.6, 160.7)
- added J18: chassis, Connector_Pin:Pin_D1.1mm_L8.5mm_W2.5mm_FlatFork, F.Cu at (154.9, 80.0)
- added R18: R, Resistor_THT:R_Axial_DIN0614_L14.3mm_D5.7mm_P20.32mm_Horizontal, F.Cu at (81.3, 112.0)
- C1: value C_Polarized -> 22u; footprint Capacitor_THT:CP_Radial_D8.0mm_P3.50mm -> Capacitor_THT:CP_Axial_L11.0mm_D6.0mm_P18.00mm_Horizontal
- C12: value C_Polarized -> 10u
- C2: value C -> 68n
- C3, C4: value C -> 82n
- C5: value C -> 220p
- C6, C8: value C -> 100n
- C7: value C -> 22n
- C9: value C -> 10n
- J1: value Screw_Terminal_01x02 -> MID Select
- J2: value Screw_Terminal_01x02 -> Input
- J3: value Screw_Terminal_01x02 -> MID Bypass
- J4: value Screw_Terminal_01x02 -> Low boost
- J5: value Screw_Terminal_01x03 -> PrePower
- J6: value Screw_Terminal_01x03 -> Volume
- J7: value Screw_Terminal_01x02 -> Hi Cut
- J8: value Screw_Terminal_01x03 -> 6N6P
- J9: value Screw_Terminal_01x01 -> OT feedback
- R1, R2: value R -> 330
- R10: value R -> 2k
- R11, R17, R3: value R -> 1k
- R12: value R -> 27k
- R13: value R -> 10k
- R14: value R -> 100k
- R15: value R -> 15k
- R16: value R -> 220
- R19, R22, R5, R6: value R -> 1Meg
- R20, R8: value R -> 12k
- R21: value R -> 330k
- R4: value R -> 68k
- R7: value R -> 18k
- R9: value R -> 390, 5W
- moved R3 72.7 mm to (128.3, 55.2), turned to -90 degrees
- moved R4 59.1 mm to (142.2, 45.7)
- moved J9 58.3 mm to (149.8, 25.4)
- moved U2 58.3 mm to (84.7, 48.9)
- moved J1 58.3 mm to (98.7, 77.5)
- moved J4 58.3 mm to (112.7, 77.5)
- moved J5 58.3 mm to (118.1, 36.8)
- moved R12 58.3 mm to (98.7, 50.9)
- moved R13 58.3 mm to (84.8, 34.9)
- moved R15 58.3 mm to (37.5, 76.8)
- moved R19 58.3 mm to (37.5, 69.8)
- moved C3 58.3 mm to (91.4, 64.8)
- moved J3 58.3 mm to (64.8, 77.5)
- moved J8 58.3 mm to (174.6, 27.9)
- moved R8 58.3 mm to (135.3, 59.0)
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Connections:
- R3 pad 1: Net-(J4-Pin_2) -> Net-(U1A-+)
- R3 pad 2: Net-(U1A-+) -> Net-(J4-Pin_2)
Routing:
- net GND2: track 0.00 -> 162.2 mm
- net Net-(D10-A): track 0.00 -> 65.2 mm
- net Net-(J16-Pin_1): track 0.00 -> 59.1 mm
- net Net-(J10-Pin_3): track 0.00 -> 49.6 mm
- net Net-(D4-A): track 0.00 -> 31.2 mm
- net Net-(D10-K): track 0.00 -> 30.2 mm
- net Net-(D3-K): track 0.00 -> 21.8 mm
- net Net-(D7-K): track 0.00 -> 19.3 mm
- net Net-(D7-A): track 0.00 -> 12.1 mm
- net Net-(D3-A): track 0.00 -> 12.1 mm
- net Net-(J8-Pin_1): track 61.2 -> 52.0 mm
- net GND: track 339.8 -> 348.4 mm
- net V++: track 108.2 -> 106.6 mm
- net Net-(D2-A): track 20.4 -> 21.6 mm
- net Net-(R1-Pad1): track 47.5 -> 46.8 mm
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Other:
- board size 165.1 x 62.9 mm -> 165.1 x 144.1 mm

Commit message: Add files via upload
Parts:
- removed C6: 100n, Capacitor_THT:C_Disc_D8.0mm_W5.0mm_P10.00mm
- added R23: 10k, Resistor_THT:R_Axial_DIN0614_L14.3mm_D5.7mm_P20.32mm_Horizontal, F.Cu at (43.2, 43.8)
- moved R21 14.2 mm to (36.2, 43.8), turned to -90 degrees
- moved R22 7.29 mm to (105.4, 71.1)
- moved C8 6.97 mm to (42.5, 34.9), turned to 180 degrees
- moved C2 6.78 mm to (112.4, 59.6)
- moved C7 6.78 mm to (112.4, 63.5)
- moved C12 4.49 mm to (95.2, 31.8)
- moved D4 3.86 mm to (42.5, 126.4)
- moved J12 3.86 mm to (26.0, 126.4)
- moved C10 3.86 mm to (62.2, 118.1)
- moved C16 3.86 mm to (83.8, 145.3)
- moved D5 3.86 mm to (32.4, 114.3)
- moved D9 3.86 mm to (32.4, 145.4)
- moved F1 3.86 mm to (72.5, 130.8)
- moved F2 3.86 mm to (72.5, 139.7)
- moved J10 3.86 mm to (90.2, 145.4)
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Connections:
- R21 pad 2: Net-(Q1-B) -> Net-(J2-Pin_2)
Routing:
- net Net-(J3-Pin_2): track 61.2 -> 75.3 mm
- net Net-(Q1-B): track 24.1 -> 10.7 mm
- net Net-(J2-Pin_2): track 7.81 -> 19.0 mm
- net Net-(Q1-E): track 31.3 -> 22.8 mm
- net Net-(R1-Pad1): track 46.8 -> 53.6 mm
- net V--: track 62.7 -> 68.3 mm
- net V++: track 106.6 -> 103.2 mm
- net Net-(U1A-+): track 26.8 -> 24.2 mm
- net Net-(U2A-+): track 21.2 -> 19.1 mm
- net Net-(D2-A): track 21.6 -> 23.5 mm
- net Net-(J6-Pin_2): track 9.13 -> 11.0 mm
- net Net-(J6-Pin_3): track 36.5 -> 38.2 mm
- net GND: track 348.4 -> 349.7 mm
- net Net-(D1-A): track 41.5 -> 42.7 mm
- net Net-(J3-Pin_1): track 58.2 -> 59.3 mm
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Other:
- board size 165.1 x 144.1 mm -> 170 x 140.9 mm

Commit message: Add files via upload
Parts:
- moved C9 2.00 mm to (107.4, 45.1)
- moved C2 1.36 mm to (112.7, 60.9)
- moved C7 1.36 mm to (112.7, 64.8)
- moved U2 1.27 mm to (84.7, 51.4)
- moved R10 1.27 mm to (77.8, 57.1)
- moved R16 1.27 mm to (84.8, 57.1)
- moved U1 0.91 mm to (121.9, 52.7)
- moved R8 0.89 mm to (136.1, 61.6)
- moved C12 0.77 mm to (95.2, 32.6)
- moved R1 0.67 mm to (149.9, 66.6)
- moved J5 0.65 mm to (117.5, 36.8)
- moved D1 0.65 mm to (160.0, 54.0)
- moved D2 0.65 mm to (160.0, 50.2)
- moved R2 0.65 mm to (149.9, 37.5)
- moved R5 0.65 mm to (170.2, 59.7)
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Routing:
- net Net-(D1-K): track 3.81 -> 0.00 mm
- net Net-(U1A-+): track 24.2 -> 27.7 mm
- net V--: track 68.3 -> 71.2 mm
- net Net-(J3-Pin_1): track 59.3 -> 56.5 mm
- net GND: track 349.7 -> 347.1 mm
- net V++: track 103.2 -> 105.7 mm
- net Net-(U1A--): track 33.1 -> 31.3 mm
- net Net-(J4-Pin_2): track 47.5 -> 46.2 mm
- net Net-(C3-Pad1): track 21.1 -> 22.4 mm
- net Net-(D2-A): track 23.5 -> 22.3 mm
- net Net-(U2A-+): track 19.1 -> 17.9 mm
- net Net-(U2B-+): track 27.4 -> 28.6 mm
- net Net-(J4-Pin_1): track 13.7 -> 12.7 mm
- net Net-(U1B--): track 11.3 -> 12.2 mm
- net Net-(R2-Pad1): track 30.9 -> 31.5 mm
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Other:
- outline, holes or cut-outs redrawn

Commit message: Add files via upload
Parts:
- added F3: Fuse, Fuse:Fuseholder_Clip-5x20mm_Keystone_3517_Inline_P23.11x6.76mm_D1.70mm_Horizontal, F.Cu at (72.8, 102.9)
- added J19: TUBE, Connector_Phoenix_MSTB:PhoenixContact_MSTBA_2,5_2-G-5,08_1x02_P5.08mm_Horizontal, F.Cu at (163.2, 29.2)
- added J20: Screw_Terminal_01x01, Connector_Pin:Pin_D1.1mm_L8.5mm_W2.5mm_FlatFork, F.Cu at (105.0, 137.8)
- added J21: Screw_Terminal_01x01, Connector_Pin:Pin_D1.1mm_L8.5mm_W2.5mm_FlatFork, F.Cu at (105.0, 128.9)
- added J22: Screw_Terminal_01x01, Connector_Pin:Pin_D1.1mm_L8.5mm_W2.5mm_FlatFork, F.Cu at (105.0, 122.6)
- C1: value 22u -> 68u/350V; footprint Capacitor_THT:CP_Axial_L11.0mm_D6.0mm_P18.00mm_Horizontal -> Capacitor_THT:CP_Radial_D16.0mm_P7.50mm
- C11, C13: footprint Capacitor_THT:CP_Radial_D12.5mm_P7.50mm -> Capacitor_THT:CP_Radial_D16.0mm_P7.50mm
- C12: footprint Capacitor_THT:CP_Radial_D12.5mm_P5.00mm -> Capacitor_THT:CP_Radial_D14.0mm_P7.50mm
- J8: value 6N6P -> chassis; footprint Connector_Phoenix_MSTB:PhoenixContact_MSTBA_2,5_3-G-5,08_1x03_P5.08mm_Horizontal -> Connector_Pin:Pin_D1.1mm_L8.5mm_W2.5mm_FlatFork
- R3, R4, R7: footprint Resistor_THT:R_Axial_DIN0614_L14.3mm_D5.7mm_P20.32mm_Horizontal -> Resistor_THT:R_Axial_DIN0614_L14.3mm_D5.7mm_P15.24mm_Horizontal
- R8: value 12k -> 10k; footprint Resistor_THT:R_Axial_DIN0614_L14.3mm_D5.7mm_P20.32mm_Horizontal -> Resistor_THT:R_Axial_DIN0614_L14.3mm_D5.7mm_P15.24mm_Horizontal
- R9: value 390, 5W -> 10k; footprint Resistor_THT:R_Axial_DIN0922_L20.0mm_D9.0mm_P30.48mm_Horizontal -> Resistor_THT:R_Axial_DIN0614_L14.3mm_D5.7mm_P15.24mm_Horizontal
- moved C1 98.1 mm to (96.4, 128.9)
- moved C15 52.6 mm to (88.3, 110.5), turned to 0 degrees
- moved J8 50.1 mm to (156.2, 74.3), turned to 90 degrees
- moved R18 50.0 mm to (52.1, 149.2), turned to 0 degrees
- moved R9 49.9 mm to (142.2, 32.4), turned to -90 degrees
- moved C10 45.5 mm to (88.9, 154.9)
- moved J10 41.4 mm to (93.3, 104.1), turned to 180 degrees
- moved D10 39.6 mm to (44.5, 113.0), turned to 90 degrees
- moved D3 37.5 mm to (43.8, 157.5), turned to 90 degrees
- moved C16 35.6 mm to (76.8, 110.5), turned to 180 degrees
- moved D6 33.9 mm to (38.1, 142.2), turned to 90 degrees
- moved D9 32.7 mm to (36.8, 113.0), turned to 90 degrees
- moved R6 32.4 mm to (168.3, 71.1), turned to 90 degrees
- moved J13 32.4 mm to (26.0, 113.0)
- moved D7 31.8 mm to (40.6, 108.0), turned to -90 degrees
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Connections:
- C1 pad 1: Net-(J8-Pin_1) -> Net-(J21-Pin_1)
- C1 pad 2: GND -> GND2
- C13 pad 2: Net-(D10-A) -> Net-(J10-Pin_2)
- C15 pad 1: Net-(D10-A) -> Net-(J10-Pin_2)
- C16 pad 1: Net-(D10-A) -> Net-(J10-Pin_2)
- J10 pad 2: Net-(D10-A) -> Net-(J10-Pin_2)
- J8 pad 1: Net-(J8-Pin_1) -> GND
- R3 pad 1: Net-(U1A-+) -> Net-(U1A--)
- R4 pad 1: Net-(U1A-+) -> Net-(U1A--)
- R8 pad 1: Net-(U1A--) -> Net-(U1B--)
- R8 pad 2: Net-(U1B--) -> Net-(R1-Pad1)
- R9 pad 1: GND -> Net-(U1B--)
- R9 pad 2: Net-(J8-Pin_1) -> Net-(R2-Pad1)
- U1 pad 3: Net-(U1A-+) -> GND
Routing:
- net GND: track 347.1 -> 3.82 mm
- net GND2: track 161.7 -> 0.00 mm
- net Net-(J10-Pin_2): track 0.00 -> 73.9 mm
- net Net-(J8-Pin_1): track 52.0 -> 0.00 mm
- net Net-(D10-A): track 65.2 -> 19.6 mm
- net Net-(U1B--): track 12.2 -> 51.2 mm
- net V++: track 105.7 -> 135.3 mm
- net Net-(U1A-+): track 27.7 -> 0.00 mm
- net V--: track 71.2 -> 95.8 mm
- net Net-(R2-Pad1): track 31.5 -> 12.6 mm
- net Net-(D1-A): track 42.7 -> 59.8 mm
- net Net-(J21-Pin_1): track 0.00 -> 14.9 mm
- net Net-(D3-A): track 12.1 -> 26.6 mm
- net Net-(D4-A): track 31.2 -> 17.1 mm
- net Net-(D7-K): track 19.3 -> 32.5 mm
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- added copper zone on F.Cu, net GND
- added copper zone on F.Cu, net GND2
Other:
- board size 170 x 140.9 mm -> 161.3 x 142.7 mm

Commit message: Add files via upload
Parts:
- moved C16 20.2 mm to (58.5, 119.1), turned to 0 degrees
- moved D7 7.73 mm to (33.0, 109.2)
- moved D8 7.73 mm to (40.6, 109.2)
- moved F2 6.61 mm to (72.8, 111.5)
- moved C11 3.51 mm to (75.9, 125.3)
- moved C13 3.29 mm to (58.9, 135.5)
- moved C15 2.68 mm to (85.7, 110.7)
- moved J10 2.54 mm to (90.8, 104.1)
- moved C14 1.98 mm to (90.6, 117.3)
- moved R18 1.91 mm to (50.2, 149.2)
- moved C10 1.27 mm to (87.6, 154.9)
- moved D10 1.02 mm to (44.5, 114.0)
- moved D9 1.02 mm to (36.8, 114.0)
- moved J13 1.02 mm to (26.0, 114.0)
- moved F3 1.02 mm to (72.8, 103.9)
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Routing:
- net Net-(J10-Pin_2): track 73.9 -> 65.4 mm
- net Net-(D7-K): track 32.5 -> 24.4 mm
- net Net-(D10-K): track 33.4 -> 25.7 mm
- net Net-(D7-A): track 18.6 -> 16.1 mm
- net Net-(J10-Pin_3): track 58.4 -> 56.5 mm
- net Net-(J16-Pin_1): track 59.5 -> 60.3 mm

Commit message: Add files via upload
Parts:
- C11, C13: footprint Capacitor_THT:CP_Radial_D16.0mm_P7.50mm -> Capacitor_THT:CP_Radial_D18.0mm_P7.50mm
- moved C13 2.55 mm to (56.4, 135.3)
- moved C11 2.48 mm to (75.2, 127.6)
- moved C16 0.25 mm to (58.5, 118.9)
Routing:
- net Net-(J10-Pin_3): track 56.5 -> 61.1 mm
- net Net-(J10-Pin_2): track 65.4 -> 63.1 mm

Commit message: Add files via upload
Parts:
- moved C16 2.97 mm to (61.5, 118.9)
- moved C8 2.80 mm to (45.9, 32.5)
- moved Q1 1.02 mm to (50.1, 34.3)
- moved J18 0.64 mm to (148.6, 73.7)
- moved J8 0.64 mm to (156.2, 73.7)
Routing:
- net Net-(J10-Pin_3): track 61.1 -> 53.9 mm
- net Net-(J10-Pin_2): track 63.1 -> 65.9 mm
- net Net-(J6-Pin_2): track 12.2 -> 14.6 mm
- net Net-(Q1-E): track 21.3 -> 19.3 mm
- net V++: track 135.3 -> 136.8 mm
- net Net-(D3-A): track 26.6 -> 27.5 mm
- net Net-(D10-K): track 25.7 -> 26.3 mm
- net Net-(Q1-B): track 10.7 -> 11.2 mm
Other:
- board text added: "P100 Exp Hybrid PRE. Rev: alpha"
- board text added: "P100 Exp Hybrid PSU. Rev: alpha"

Commit message: Add files via upload
Parts:
- removed D10, D4, D5, D6, D7, D8, D9: 1N4001, Diode_THT:D_DO-41_SOD81_P10.16mm_Horizontal
- removed J17: center tap, Connector_Pin:Pin_D1.1mm_L8.5mm_W2.5mm_FlatFork
- added D11: B40C2300-1500B, Diode_THT:Diode_Bridge_19.0x3.5x10.0mm_P5.0mm, F.Cu at (38.7, 107.5)
- added R24: 0, Resistor_THT:R_Axial_DIN0204_L3.6mm_D1.6mm_P5.08mm_Horizontal, F.Cu at (46.4, 26.0)
- D3: value 1N4001 -> B40C2300-1500B; footprint Diode_THT:D_DO-41_SOD81_P10.16mm_Horizontal -> Diode_THT:Diode_Bridge_19.0x3.5x10.0mm_P5.0mm
- Q1: footprint Package_TO_SOT_THT:TO-92L_Inline_Wide -> Package_TO_SOT_THT:TO-92S_Wide
- R20: footprint Resistor_THT:R_Axial_DIN0614_L14.3mm_D5.7mm_P20.32mm_Horizontal -> Resistor_THT:R_Axial_DIN0414_L11.9mm_D4.5mm_P15.24mm_Horizontal
- moved J8 129.8 mm to (35.5, 26.0), turned to 180 degrees
- moved R5 26.8 mm to (161.3, 73.7), turned to 180 degrees
- moved D3 25.8 mm to (38.7, 132.2), turned to -90 degrees
- moved R9 25.0 mm to (119.4, 42.5)
- moved C16 21.7 mm to (73.7, 101.0), turned to -90 degrees
- moved J18 14.5 mm to (161.3, 80.6), turned to 0 degrees
- moved J14 12.7 mm to (31.8, 112.5)
- moved J12 11.7 mm to (31.8, 137.2)
- moved J11 11.0 mm to (31.8, 147.2)
- moved C13 11.0 mm to (50.9, 125.7), turned to 0 degrees
- moved J13 10.2 mm to (31.8, 122.5)
- moved D1 8.63 mm to (165.6, 34.9)
- moved C4 7.72 mm to (90.2, 43.3)
- moved R8 7.65 mm to (133.3, 42.5)
- moved R2 7.24 mm to (141.0, 42.5)
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Connections:
- D3 pad 1: Net-(D3-K) -> GND2
- D3 pad 2: Net-(D3-A) -> Net-(J12-Pin_1)
- F1 pad 2: Net-(D3-K) -> Net-(D3-+)
- J11 pad 1: Net-(D3-A) -> Net-(J11-Pin_1)
- J12 pad 1: Net-(D4-A) -> Net-(J12-Pin_1)
Routing:
- net GND: track 3.82 -> 119.5 mm
- net GND2: track 0.00 -> 51.7 mm
- net Net-(D3-+): track 0.00 -> 34.8 mm
- net Net-(D3-A): track 27.5 -> 0.00 mm
- net Net-(R2-Pad1): track 12.6 -> 37.9 mm
- net Net-(R1-Pad1): track 53.7 -> 32.4 mm
- net Net-(J14-Pin_1): track 26.3 -> 6.99 mm
- net Net-(D3-K): track 18.1 -> 0.00 mm
- net Net-(D4-A): track 17.1 -> 0.00 mm
- net Net-(U1B--): track 51.2 -> 37.4 mm
- net Net-(D1-A): track 59.8 -> 47.2 mm
- net Net-(J3-Pin_2): track 76.0 -> 66.0 mm
- net Net-(J13-Pin_1): track 16.1 -> 6.99 mm
- net Net-(J10-Pin_3): track 53.9 -> 62.1 mm
- net Net-(J4-Pin_2): track 42.3 -> 50.0 mm
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- added copper zone on B.Cu, net GND3
Other:
- board size 161.3 x 142.7 mm -> 156.3 x 142.7 mm
