File: KiCad/6N6P_hybrid.kicad_pcb (KiCad board)
At the start: 2 copper layers, 156.3 x 142.7 mm, 70 parts, among them J1 MID Select, J10 Screw_Terminal_01x03, J11 Screw_Terminal_01x01, J12 Screw_Terminal_01x01, J13 Screw_Terminal_01x01, J14 Screw_Terminal_01x01, J15 PSU ground, J16 Screw_Terminal_01x01, J18 chassis, J19 TUBE, J2 Input, J20 Screw_Terminal_01x01, J21 Screw_Terminal_01x01, J22 Screw_Terminal_01x01, J3 MID Bypass, J4 Low boost, J5 PrePower, J6 Volume, J7 Hi Cut, J8 chassis, J9 OT feedback, Q1 BC107, U1 LTC1151CN8, U2 LTC1151CN8

Commit message: Add files via upload
Parts:
- removed J20, J21: Screw_Terminal_01x01, Connector_Pin:Pin_D1.1mm_L8.5mm_W2.5mm_FlatFork
- added R25: R, Resistor_THT:R_Axial_DIN0617_L17.0mm_D6.0mm_P25.40mm_Horizontal, F.Cu at (100.1, 144.8)
- moved C14 24.4 mm to (63.6, 118.7), turned to 0 degrees
- moved C1 7.78 mm to (89.4, 122.6)
- moved J16 5.10 mm to (106.2, 141.7), turned to 0 degrees
- moved J22 4.57 mm to (106.2, 122.4)
- moved J15 2.63 mm to (100.1, 110.7)
- moved F1 2.14 mm to (67.7, 157.2)
- moved C11 2.03 mm to (70.5, 127.6)
- moved C13 1.90 mm to (49.0, 125.7)
- moved C10 1.31 mm to (83.8, 154.3)
Routing:
- net Net-(J16-Pin_1): track 59.3 -> 69.2 mm
- net Net-(J10-Pin_3): track 62.1 -> 56.5 mm
- net Net-(J22-Pin_1): track 14.4 -> 19.1 mm
- net GND2: track 51.7 -> 49.5 mm
- net Net-(J10-Pin_2): track 67.3 -> 66.6 mm
Other:
- outline, holes or cut-outs redrawn
