File: KiCad/6N6P_hybrid.kicad_sch (KiCad schematic)
At the start: 45 parts, among them J1 Screw_Terminal_01x02, J2 Screw_Terminal_01x02, J3 Screw_Terminal_01x02, J4 Screw_Terminal_01x02, J5 Screw_Terminal_01x03, J6 Screw_Terminal_01x03, J7 Screw_Terminal_01x02, J8 Screw_Terminal_01x03, J9 Screw_Terminal_01x01, Q1 BC107, U1 LTC1151CN8, U2 LTC1151CN8

Commit message: Add files via upload
Parts:
- added J18: chassis, Connector_Pin:Pin_D1.1mm_L8.5mm_W2.5mm_FlatFork, symbol Connector:Screw_Terminal_01x01
- C1: footprint Capacitor_THT:CP_Radial_D8.0mm_P3.50mm -> Capacitor_THT:CP_Axial_L11.0mm_D6.0mm_P18.00mm_Horizontal
- C5: value C -> 220p
- J1: value Screw_Terminal_01x02 -> MID Select
- J2: value Screw_Terminal_01x02 -> Input
- J3: value Screw_Terminal_01x02 -> MID Bypass
- J4: value Screw_Terminal_01x02 -> Low boost
- J5: value Screw_Terminal_01x03 -> PrePower
- J6: value Screw_Terminal_01x03 -> Volume
- J7: value Screw_Terminal_01x02 -> Hi Cut
- J8: value Screw_Terminal_01x03 -> 6N6P
- J9: value Screw_Terminal_01x01 -> OT feedback
Connections:
- net GND: now also J18.1 (Pin_1)
Other:
- removed sheet Equaliser
Changed lines of the file:
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@@
+    (stroke (width 0) (type default))
+  )
+  (wire (pts (xy 206.375 82.55) (xy 204.47 82.55))
     (stroke (width 0) (type default))
   )
@@
   )
   (wire (pts (xy 27.94 87.63) (xy 27.94 93.98))
+    (stroke (width 0) (type default))
+  )
+  (wire (pts (xy 204.47 82.55) (xy 204.47 86.995))
     (stroke (width 0) (type default))
   )
@@
       (effects (font (size 1.27 1.27)) (justify left))
     )
-    (property "Value" "Screw_Terminal_01x03" (at 116.84 56.515 0)
+    (property "Value" "PrePower" (at 116.84 56.515 0)
       (effects (font (size 1.27 1.27)) (justify left))
     )
@@
       (effects (font (size 1.27 1.27)))
     )
-    (property "Value" "Screw_Terminal_01x03" (at 77.47 100.33 0)
+    (property "Value" "Volume" (at 77.47 100.33 0)
       (effects (font (size 1.27 1.27)))
     )
@@
       (effects (font (size 1.27 1.27)) (justify left))
     )
-    (property "Value" "Screw_Terminal_01x01" (at 220.98 109.855 0)
+    (property "Value" "OT feedback" (at 220.98 109.855 0)
       (effects (font (size 1.27 1.27)) (justify left))
     )
@@
       (effects (font (size 1.27 1.27)) (justify left))
     )
-    (property "Value" "Screw_Terminal_01x02" (at 129.54 79.375 90)
+    (property "Value" "MID Bypass" (at 129.54 79.375 90)
       (effects (font (size 1.27 1.27)) (justify left))
     )
@@
     )
   )
+  (symbol (lib_id "Connector:Screw_Terminal_01x01") (at 211.455 82.55 0) (unit 1)
+    (in_bom yes) (on_board yes) (dnp no) (fields_autoplaced)
+    (property "Reference" "J18" (at 214.63 81.915 0)
+      (effects (font (size 1.27 1.27)) (justify left))
+    )
+    (property "Value" "chassis" (at 214.63 84.455 0)
+      (effects (font (size 1.27 1.27)) (justify left))
+    )
+    (property "Footprint" "Connector_Pin:Pin_D1.1mm_L8.5mm_W2.5mm_FlatFork" (at 211.455 82.55 0)
+      (effects (font (size 1.27 1.27)) hide)
+    )
+    (property "Datasheet" "~" (at 211.455 82.55 0)
+      (effects (font (size 1.27 1.27)) hide)
+    )
+    (pin "1")
+    (instances
+      (project "6N6P_hybrid"
+        (path "/ef50db11-0c56-48df-b02f-5ef4676a3739"
+          (reference "J18") (unit 1)
+        )
+      )
+    )
+  )
   (symbol (lib_id "Device:R") (at 43.18 96.52 180) (unit 1)
     (in_bom yes) (on_board yes) (dnp no) (fields_autoplaced)
@@
       (effects (font (size 1.27 1.27)))
     )
-    (property "Footprint" "Capacitor_THT:CP_Radial_D8.0mm_P3.50mm" (at 233.68 136.8552 0)
+    (property "Footprint" "Capacitor_THT:CP_Axial_L11.0mm_D6.0mm_P18.00mm_Horizontal" (at 233.68 136.8552 0)
       (effects (font (size 1.27 1.27)) hide)
     )
@@
       (effects (font (size 1.27 1.27)))
     )
-    (property "Value" "Screw_Terminal_01x03" (at 259.08 130.81 0)
+    (property "Value" "6N6P" (at 259.08 130.81 0)
       (effects (font (size 1.27 1.27)))
     )
@@
       (effects (font (size 1.27 1.27)))
     )
-    (property "Value" "C" (at 88.9 115.57 90)
+    (property "Value" "220p" (at 88.9 115.57 90)
       (effects (font (size 1.27 1.27)))
     )
@@
       (effects (font (size 1.27 1.27)))
     )
-    (property "Value" "Screw_Terminal_01x02" (at 22.86 99.06 0)
-      (effects (font (size 1.27 1.27)) hide)
+    (property "Value" "Input" (at 22.86 99.06 0)
+      (effects (font (size 1.27 1.27)))
     )
     (property "Footprint" "Connector_Phoenix_MSTB:PhoenixContact_MSTBA_2,5_2-G-5,08_1x02_P5.08mm_Horizontal" (at 22.86 96.52 0)
@@
       (effects (font (size 1.27 1.27)) (justify left))
     )
-    (property "Value" "Screw_Terminal_01x02" (at 161.29 71.755 90)
+    (property "Value" "Low boost" (at 161.29 71.755 90)
       (effects (font (size 1.27 1.27)) (justify left))
     )
@@
       (effects (font (size 1.27 1.27)))
     )
-    (property "Value" "Screw_Terminal_01x02" (at 115.57 153.67 0)
+    (property "Value" "MID Select" (at 115.57 153.67 0)
       (effects (font (size 1.27 1.27)))
     )
@@
       (effects (font (size 1.27 1.27)))
     )
-    (property "Value" "Screw_Terminal_01x02" (at 90.17 127 0)
-      (effects (font (size 1.27 1.27)) hide)
+    (property "Value" "Hi Cut" (at 90.17 127 0)
+      (effects (font (size 1.27 1.27)))
     )
     (property "Footprint" "Connector_Phoenix_MSTB:PhoenixContact_MSTBA_2,5_2-G-5,08_1x02_P5.08mm_Horizontal" (at 90.17 129.54 0)
@@
         (path "/ef50db11-0c56-48df-b02f-5ef4676a3739"
           (reference "J7") (unit 1)
+        )
+      )
+    )
+  )
+  (symbol (lib_id "power:GND") (at 204.47 86.995 0) (unit 1)
+    (in_bom yes) (on_board yes) (dnp no) (fields_autoplaced)
+    (property "Reference" "#PWR015" (at 204.47 93.345 0)
+      (effects (font (size 1.27 1.27)) hide)
+    )
+    (property "Value" "GND" (at 204.47 92.075 0)
+      (effects (font (size 1.27 1.27)))
+    )
+    (property "Footprint" "" (at 204.47 86.995 0)
+      (effects (font (size 1.27 1.27)) hide)
+    )
+    (property "Datasheet" "" (at 204.47 86.995 0)
+      (effects (font (size 1.27 1.27)) hide)
+    )
+    (pin "1")
+    (instances
+      (project "6N6P_hybrid"
+        (path "/ef50db11-0c56-48df-b02f-5ef4676a3739"
+          (reference "#PWR015") (unit 1)
         )
       )
@@
     )
   )
-  (sheet (at 320.04 66.04) (size 162.56 138.43) (fields_autoplaced)
+  (sheet (at 207.01 19.05) (size 38.1 30.48) (fields_autoplaced)
     (stroke (width 0.1524) (type solid))
     (fill (color 0 0 0 0.0000))
-    (property "Sheetname" "PSU" (at 320.04 65.3284 0)
+    (property "Sheetname" "PSU" (at 207.01 18.3384 0)
       (effects (font (size 1.27 1.27)) (justify left bottom))
     )
-    (property "Sheetfile" "psu.kicad_sch" (at 320.04 205.0546 0)
+    (property "Sheetfile" "psu.kicad_sch" (at 207.01 50.1146 0)
       (effects (font (size 1.27 1.27)) (justify left top))
     )
@@
       )
     )
-  )
-  (sheet (at 317.5 2.54) (size 90.17 50.8) (fields_autoplaced)
-    (stroke (width 0.1524) (type solid))
-    (fill (color 0 0 0 0.0000))
-    (property "Sheetname" "Equaliser" (at 317.5 1.8284 0)
-      (effects (font (size 1.27 1.27)) (justify left bottom))
-    )
-    (property "Sheetfile" "euqliser.kicad_sch" (at 317.5 53.9246 0)
-      (effects (font (size 1.27 1.27)) (justify left top))
-    )
-    (instances
-      (project "6N6P_hybrid"
-        (path "/ef50db11-0c56-48df-b02f-5ef4676a3739" (page "3"))
-      )
-    )

Commit message: Add files via upload
Parts:
- removed C6: 100n, Capacitor_THT:C_Disc_D8.0mm_W5.0mm_P10.00mm, symbol Device:C
- added R23: 10k, Resistor_THT:R_Axial_DIN0614_L14.3mm_D5.7mm_P20.32mm_Horizontal, symbol Device:R
Connections:
- net at J2.2 (Pin_2): now also R21.2, R23.2
- net at Q1.2 (B): now also R23.1; no longer R21.2
Other:
- added sheet Equaliser (equaliser.kicad_sch)
- moved on the sheet: R21
Changed lines of the file:
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@@
   (junction (at 223.52 153.67) (diameter 0) (color 0 0 0 0)
   )
+  (junction (at 35.56 87.63) (diameter 0) (color 0 0 0 0)
+  )
   (junction (at 194.31 124.46) (diameter 0) (color 0 0 0 0)
   )
@@
   (junction (at 210.82 124.46) (diameter 0) (color 0 0 0 0)
   )
-  (junction (at 43.18 87.63) (diameter 0) (color 0 0 0 0)
-  )
   (junction (at 54.61 93.98) (diameter 0) (color 0 0 0 0)
   )
@@
   (junction (at 223.52 142.24) (diameter 0) (color 0 0 0 0)
   )
-  (junction (at 163.83 74.93) (diameter 0) (color 0 0 0 0)
-  )
   (junction (at 171.45 107.95) (diameter 0) (color 0 0 0 0)
   )
   (junction (at 95.25 39.37) (diameter 0) (color 0 0 0 0)
   )
-  (wire (pts (xy 27.94 87.63) (xy 31.75 87.63))
+  (wire (pts (xy 27.94 87.63) (xy 35.56 87.63))
     (stroke (width 0) (type default))
   )
@@
     (stroke (width 0) (type default))
   )
+  (wire (pts (xy 35.56 87.63) (xy 37.465 87.63))
+    (stroke (width 0) (type default))
+  )
   (wire (pts (xy 241.3 135.89) (xy 243.84 135.89))
     (stroke (width 0) (type default))
@@
     (stroke (width 0) (type default))
   )
-  (wire (pts (xy 164.465 74.93) (xy 163.83 74.93))
-    (stroke (width 0) (type default))
-  )
   (wire (pts (xy 223.52 142.24) (xy 223.52 143.51))
     (stroke (width 0) (type default))
@@
     (stroke (width 0) (type default))
   )
-  (wire (pts (xy 43.18 87.63) (xy 43.18 92.71))
+  (wire (pts (xy 35.56 87.63) (xy 35.56 92.71))
     (stroke (width 0) (type default))
   )
@@
     (stroke (width 0) (type default))
   )
+  (wire (pts (xy 45.085 87.63) (xy 46.99 87.63))
+    (stroke (width 0) (type default))
+  )
   (wire (pts (xy 223.52 142.24) (xy 233.68 142.24))
     (stroke (width 0) (type default))
@@
     (stroke (width 0) (type default))
   )
+  (wire (pts (xy 158.75 74.93) (xy 163.83 74.93))
+    (stroke (width 0) (type default))
+  )
   (wire (pts (xy 158.75 83.82) (xy 161.29 83.82))
     (stroke (width 0) (type default))
   )
-  (wire (pts (xy 43.18 100.33) (xy 43.18 104.14))
+  (wire (pts (xy 35.56 100.33) (xy 35.56 104.14))
     (stroke (width 0) (type default))
   )
@@
     (stroke (width 0) (type default))
   )
-  (wire (pts (xy 163.83 74.93) (xy 158.75 74.93))
-    (stroke (width 0) (type default))
-  )
   (wire (pts (xy 223.52 124.46) (xy 223.52 127))
     (stroke (width 0) (type default))
@@
     (stroke (width 0) (type default))
   )
-  (wire (pts (xy 43.18 87.63) (xy 46.99 87.63))
-    (stroke (width 0) (type default))
-  )
   (wire (pts (xy 205.74 153.67) (xy 210.82 153.67))
     (stroke (width 0) (type default))
@@
   )
   (wire (pts (xy 171.45 74.93) (xy 171.45 83.82))
-    (stroke (width 0) (type default))
-  )
-  (wire (pts (xy 39.37 87.63) (xy 43.18 87.63))
     (stroke (width 0) (type default))
   )
@@
     )
   )
-  (symbol (lib_id "Device:C") (at 35.56 87.63 90) (unit 1)
-    (in_bom yes) (on_board yes) (dnp no) (fields_autoplaced)
-    (property "Reference" "C6" (at 35.56 81.28 90)
-      (effects (font (size 1.27 1.27)))
-    )
-    (property "Value" "100n" (at 35.56 83.82 90)
-      (effects (font (size 1.27 1.27)))
-    )
-    (property "Footprint" "Capacitor_THT:C_Disc_D8.0mm_W5.0mm_P10.00mm" (at 39.37 86.6648 0)
-      (effects (font (size 1.27 1.27)) hide)
-    )
-    (property "Datasheet" "~" (at 35.56 87.63 0)
-      (effects (font (size 1.27 1.27)) hide)
-    )
-    (pin "1")
-    (pin "2")
-    (instances
-      (project "6N6P_hybrid"
-        (path "/ef50db11-0c56-48df-b02f-5ef4676a3739"
-          (reference "C6") (unit 1)
-        )
-      )
-    )
-  )
   (symbol (lib_id "power:GND") (at 81.28 138.43 0) (unit 1)
     (in_bom yes) (on_board yes) (dnp no) (fields_autoplaced)
@@
     )
   )
-  (symbol (lib_id "Device:R") (at 43.18 96.52 180) (unit 1)
-    (in_bom yes) (on_board yes) (dnp no) (fields_autoplaced)
-    (property "Reference" "R21" (at 45.72 95.885 0)
+  (symbol (lib_id "Device:R") (at 35.56 96.52 180) (unit 1)
+    (in_bom yes) (on_board yes) (dnp no) (fields_autoplaced)
+    (property "Reference" "R21" (at 38.1 95.885 0)
       (effects (font (size 1.27 1.27)) (justify right))
     )
-    (property "Value" "330k" (at 45.72 98.425 0)
+    (property "Value" "330k" (at 38.1 98.425 0)
       (effects (font (size 1.27 1.27)) (justify right))
     )
-    (property "Footprint" "Resistor_THT:R_Axial_DIN0614_L14.3mm_D5.7mm_P20.32mm_Horizontal" (at 44.958 96.52 90)
-      (effects (font (size 1.27 1.27)) hide)
-    )
-    (property "Datasheet" "~" (at 43.18 96.52 0)
+    (property "Footprint" "Resistor_THT:R_Axial_DIN0614_L14.3mm_D5.7mm_P20.32mm_Horizontal" (at 37.338 96.52 90)
+      (effects (font (size 1.27 1.27)) hide)
+    )
+    (property "Datasheet" "~" (at 35.56 96.52 0)
       (effects (font (size 1.27 1.27)) hide)
     )
@@
     )
   )
-  (symbol (lib_id "power:GND") (at 43.18 104.14 0) (unit 1)
-    (in_bom yes) (on_board yes) (dnp no) (fields_autoplaced)
-    (property "Reference" "#PWR05" (at 43.18 110.49 0)
-      (effects (font (size 1.27 1.27)) hide)
-    )
-    (property "Value" "GND" (at 43.18 109.22 0)
-      (effects (font (size 1.27 1.27)))
-    )
-    (property "Footprint" "" (at 43.18 104.14 0)
-      (effects (font (size 1.27 1.27)) hide)
-    )
-    (property "Datasheet" "" (at 43.18 104.14 0)
+  (symbol (lib_id "power:GND") (at 35.56 104.14 0) (unit 1)
+    (in_bom yes) (on_board yes) (dnp no) (fields_autoplaced)
+    (property "Reference" "#PWR05" (at 35.56 110.49 0)
+      (effects (font (size 1.27 1.27)) hide)
+    )
+    (property "Value" "GND" (at 35.56 109.22 0)
+      (effects (font (size 1.27 1.27)))
+    )
+    (property "Footprint" "" (at 35.56 104.14 0)
+      (effects (font (size 1.27 1.27)) hide)
+    )
+    (property "Datasheet" "" (at 35.56 104.14 0)
       (effects (font (size 1.27 1.27)) hide)
     )
@@
     )
   )
+  (symbol (lib_id "Device:R") (at 41.275 87.63 270) (unit 1)
+    (in_bom yes) (on_board yes) (dnp no) (fields_autoplaced)
+    (property "Reference" "R23" (at 41.275 82.55 90)
+      (effects (font (size 1.27 1.27)))
+    )
+    (property "Value" "10k" (at 41.275 85.09 90)
+      (effects (font (size 1.27 1.27)))
+    )
+    (property "Footprint" "Resistor_THT:R_Axial_DIN0614_L14.3mm_D5.7mm_P20.32mm_Horizontal" (at 41.275 85.852 90)
+      (effects (font (size 1.27 1.27)) hide)
+    )
+    (property "Datasheet" "~" (at 41.275 87.63 0)
+      (effects (font (size 1.27 1.27)) hide)
+    )
+    (pin "1")
+    (pin "2")
+    (instances
+      (project "6N6P_hybrid"
+        (path "/ef50db11-0c56-48df-b02f-5ef4676a3739"
+          (reference "R23") (unit 1)
+        )
+      )
+    )
+  )
   (symbol (lib_id "Device:R") (at 223.52 147.32 0) (unit 1)
     (in_bom yes) (on_board yes) (dnp no) (fields_autoplaced)
@@
       )
     )
+  )
+  (sheet (at 27.305 154.94) (size 32.385 21.59) (fields_autoplaced)
+    (stroke (width 0.1524) (type solid))
+    (fill (color 0 0 0 0.0000))
+    (property "Sheetname" "Equaliser" (at 27.305 154.2284 0)
+      (effects (font (size 1.27 1.27)) (justify left bottom))
+    )
+    (property "Sheetfile" "equaliser.kicad_sch" (at 27.305 177.1146 0)
+      (effects (font (size 1.27 1.27)) (justify left top))
+    )
+    (property "Field2" "" (at 27.305 154.94 0)
+      (effects (font (size 1.27 1.27)) hide)
+    )
+    (instances
+      (project "6N6P_hybrid"
+        (path "/ef50db11-0c56-48df-b02f-5ef4676a3739" (page "3"))
+      )
+    )

Commit message: Add files via upload
Parts:
- removed C1: 22u, Capacitor_THT:CP_Axial_L11.0mm_D6.0mm_P18.00mm_Horizontal, symbol Device:C_Polarized
- removed J8: 6N6P, Connector_Phoenix_MSTB:PhoenixContact_MSTBA_2,5_3-G-5,08_1x03_P5.08mm_Horizontal, symbol Connector:Screw_Terminal_01x03
- added J19: TUBE, Connector_Phoenix_MSTB:PhoenixContact_MSTBA_2,5_2-G-5,08_1x02_P5.08mm_Horizontal, symbol Connector:Screw_Terminal_01x02
- added J8: chassis, Connector_Pin:Pin_D1.1mm_L8.5mm_W2.5mm_FlatFork, symbol Connector:Screw_Terminal_01x01
- C12: footprint Capacitor_THT:CP_Radial_D12.5mm_P5.00mm -> Capacitor_THT:CP_Radial_D14.0mm_P7.50mm
- R3, R4, R7: footprint Resistor_THT:R_Axial_DIN0614_L14.3mm_D5.7mm_P20.32mm_Horizontal -> Resistor_THT:R_Axial_DIN0614_L14.3mm_D5.7mm_P15.24mm_Horizontal
- R8: value 12k -> 10k; footprint Resistor_THT:R_Axial_DIN0614_L14.3mm_D5.7mm_P20.32mm_Horizontal -> Resistor_THT:R_Axial_DIN0614_L14.3mm_D5.7mm_P15.24mm_Horizontal
- R9: value 390, 5W -> 10k; footprint Resistor_THT:R_Axial_DIN0922_L20.0mm_D9.0mm_P30.48mm_Horizontal -> Resistor_THT:R_Axial_DIN0614_L14.3mm_D5.7mm_P15.24mm_Horizontal
Connections:
- net GND: now also U1.3 (+), J8.1 (Pin_1); no longer R9.1
- net at R3.1, R4.1: now also R7.1, U1.2 (-); no longer U1.3 (+)
- net at U1.6 (-): now also R8.1, R9.1; no longer R8.2
- net at R2.1, U1.7: now also R9.2
- net at D2.2 (A), R2.2, R6.2: now also J19.1 (Pin_1)
- net at R1.1, R7.2, U1.1: now also R8.2
- net at D1.2 (A), R1.2, R5.1: now also J19.2 (Pin_2)
Other:
- note added: "18V zeners to protect 6N6P from working with grid current"
- note removed: "15V zeners to protect 6N6P from working with grid current"
- moved on the sheet: R8

Commit message: Add files via upload
Parts:
- added R24: 0, Resistor_THT:R_Axial_DIN0204_L3.6mm_D1.6mm_P5.08mm_Horizontal, symbol Device:R
- Q1: footprint Package_TO_SOT_THT:TO-92L_Inline_Wide -> Package_TO_SOT_THT:TO-92S_Wide
- R20: footprint Resistor_THT:R_Axial_DIN0614_L14.3mm_D5.7mm_P20.32mm_Horizontal -> Resistor_THT:R_Axial_DIN0414_L11.9mm_D4.5mm_P15.24mm_Horizontal
Connections:
- net GND: now also R24.1
- new net GND3: R24.2
Changed lines of the file:
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@@
+    (stroke (width 0) (type default))
+  )
+  (wire (pts (xy 250.825 72.39) (xy 250.825 81.915))
     (stroke (width 0) (type default))
   )
@@
     (stroke (width 0) (type default))
   )
+  (wire (pts (xy 240.665 84.455) (xy 240.665 87.63))
+    (stroke (width 0) (type default))
+  )
   (wire (pts (xy 171.45 145.415) (xy 182.88 145.415))
     (stroke (width 0) (type default))
@@
     (stroke (width 0) (type default))
   )
+  (wire (pts (xy 240.665 72.39) (xy 240.665 76.835))
+    (stroke (width 0) (type default))
+  )
   (wire (pts (xy 171.45 106.68) (xy 171.45 107.95))
     (stroke (width 0) (type default))
@@
   )
   (wire (pts (xy 107.95 96.52) (xy 107.95 106.68))
+    (stroke (width 0) (type default))
+  )
+  (wire (pts (xy 240.665 72.39) (xy 250.825 72.39))
     (stroke (width 0) (type default))
   )
@@
         (path "/ef50db11-0c56-48df-b02f-5ef4676a3739"
           (reference "R10") (unit 1)
+        )
+      )
+    )
+  )
+  (symbol (lib_id "power:GND") (at 240.665 87.63 0) (unit 1)
+    (in_bom yes) (on_board yes) (dnp no) (fields_autoplaced)
+    (property "Reference" "#PWR018" (at 240.665 93.98 0)
+      (effects (font (size 1.27 1.27)) hide)
+    )
+    (property "Value" "GND" (at 240.665 92.71 0)
+      (effects (font (size 1.27 1.27)))
+    )
+    (property "Footprint" "" (at 240.665 87.63 0)
+      (effects (font (size 1.27 1.27)) hide)
+    )
+    (property "Datasheet" "" (at 240.665 87.63 0)
+      (effects (font (size 1.27 1.27)) hide)
+    )
+    (pin "1")
+    (instances
+      (project "6N6P_hybrid"
+        (path "/ef50db11-0c56-48df-b02f-5ef4676a3739"
+          (reference "#PWR018") (unit 1)
         )
       )
@@
       (effects (font (size 1.27 1.27)) (justify left))
     )
-    (property "Footprint" "Resistor_THT:R_Axial_DIN0614_L14.3mm_D5.7mm_P20.32mm_Horizontal" (at 79.502 130.81 90)
+    (property "Footprint" "Resistor_THT:R_Axial_DIN0414_L11.9mm_D4.5mm_P15.24mm_Horizontal" (at 79.502 130.81 90)
       (effects (font (size 1.27 1.27)) hide)
     )
@@
     )
   )
+  (symbol (lib_id "power:GND3") (at 250.825 81.915 0) (unit 1)
+    (in_bom yes) (on_board yes) (dnp no) (fields_autoplaced)
+    (property "Reference" "#PWR019" (at 250.825 88.265 0)
+      (effects (font (size 1.27 1.27)) hide)
+    )
+    (property "Value" "GND3" (at 250.825 86.36 0)
+      (effects (font (size 1.27 1.27)))
+    )
+    (property "Footprint" "" (at 250.825 81.915 0)
+      (effects (font (size 1.27 1.27)) hide)
+    )
+    (property "Datasheet" "" (at 250.825 81.915 0)
+      (effects (font (size 1.27 1.27)) hide)
+    )
+    (pin "1")
+    (instances
+      (project "6N6P_hybrid"
+        (path "/ef50db11-0c56-48df-b02f-5ef4676a3739"
+          (reference "#PWR019") (unit 1)
+        )
+      )
+    )
+  )
   (symbol (lib_id "Device:C_Polarized") (at 83.82 53.34 0) (unit 1)
     (in_bom yes) (on_board yes) (dnp no) (fields_autoplaced)
@@
     )
   )
+  (symbol (lib_id "Device:R") (at 240.665 80.645 180) (unit 1)
+    (in_bom yes) (on_board yes) (dnp no) (fields_autoplaced)
+    (property "Reference" "R24" (at 242.57 80.01 0)
+      (effects (font (size 1.27 1.27)) (justify right))
+    )
+    (property "Value" "0" (at 242.57 82.55 0)
+      (effects (font (size 1.27 1.27)) (justify right))
+    )
+    (property "Footprint" "Resistor_THT:R_Axial_DIN0204_L3.6mm_D1.6mm_P5.08mm_Horizontal" (at 242.443 80.645 90)
+      (effects (font (size 1.27 1.27)) hide)
+    )
+    (property "Datasheet" "~" (at 240.665 80.645 0)
+      (effects (font (size 1.27 1.27)) hide)
+    )
+    (pin "1")
+    (pin "2")
+    (instances
+      (project "6N6P_hybrid"
+        (path "/ef50db11-0c56-48df-b02f-5ef4676a3739"
+          (reference "R24") (unit 1)
+        )
+      )
+    )
+  )
   (symbol (lib_id "Transistor_BJT:BC107") (at 52.07 87.63 0) (unit 1)
     (in_bom yes) (on_board yes) (dnp no) (fields_autoplaced)
@@
       (effects (font (size 1.27 1.27)) (justify left))
     )
-    (property "Footprint" "Package_TO_SOT_THT:TO-92L_Inline_Wide" (at 57.15 89.535 0)
+    (property "Footprint" "Package_TO_SOT_THT:TO-92S_Wide" (at 57.15 89.535 0)
       (effects (font (size 1.27 1.27) italic) (justify left) hide)
     )
