File: KiCad/psu.kicad_sch (KiCad schematic)
At the start: 21 parts, among them J2 Screw_Terminal_01x02, J8 Screw_Terminal_01x03, J9 Screw_Terminal_01x01

Commit message: Add files via upload
Parts:
- removed J2: Screw_Terminal_01x02, Connector_Phoenix_MSTB:PhoenixContact_MSTBA_2,5_2-G-5,08_1x02_P5.08mm_Horizontal, symbol Connector:Screw_Terminal_01x02
- added F1, F2: Fuse, Fuse:Fuseholder_Clip-5x20mm_Keystone_3517_Inline_P23.11x6.76mm_D1.70mm_Horizontal, symbol Device:Fuse
- added J9: center tap, Connector_Pin:Pin_D1.1mm_L8.5mm_W2.5mm_FlatFork, symbol Connector:Screw_Terminal_01x01
- added J9: PSU ground, Connector_Pin:Pin_D1.1mm_L8.5mm_W2.5mm_FlatFork, symbol Connector:Screw_Terminal_01x01
- added J9: Screw_Terminal_01x01, Connector_Pin:Pin_D1.1mm_L8.5mm_W2.5mm_FlatFork, symbol Connector:Screw_Terminal_01x01
Connections:
- net at C11.1, C9.2, C9.2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: now also F2.1; no longer D7.1 (K), D8.1 (K)
- net at C10.1, R11.2: now also F1.1, J9.1 (Pin_1); no longer D3.1 (K), D4.1 (K)
- net GND renamed GND2
- net GND2: now also J9.1 (Pin_1), J9.1 (Pin_1)
- new net: D7.1 (K), D8.1 (K), F2.2
- new net: D3.1 (K), D4.1 (K), F1.2

Commit message: Add files via upload
Parts:
- added C1: 68u/350V, Capacitor_THT:CP_Radial_D16.0mm_P7.50mm, symbol Device:C_Polarized
- added F3: Fuse, Fuse:Fuseholder_Clip-5x20mm_Keystone_3517_Inline_P23.11x6.76mm_D1.70mm_Horizontal, symbol Device:Fuse
- added J9 (x3): Screw_Terminal_01x01, Connector_Pin:Pin_D1.1mm_L8.5mm_W2.5mm_FlatFork, symbol Connector:Screw_Terminal_01x01
- C11, C13: footprint Capacitor_THT:CP_Radial_D12.5mm_P7.50mm -> Capacitor_THT:CP_Radial_D16.0mm_P7.50mm
Connections:
- net GND2: now also C1.2
- net at C13.2, C9.1, C9.1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: now also F3.1; no longer D10.2 (A), D9.2 (A)
- net at C10.1, F1.1, J9.1 (Pin_1)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: now also J9.1 (Pin_1)
- new net: D10.2 (A), D9.2 (A), F3.2
- new net: C1.1, J9.1 (Pin_1), J9.1 (Pin_1)
Other:
- moved on the sheet: J9

Commit message: Add files via upload
Parts:
- C11, C13: footprint Capacitor_THT:CP_Radial_D16.0mm_P7.50mm -> Capacitor_THT:CP_Radial_D18.0mm_P7.50mm
Changed lines of the file:
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@@
       (effects (font (size 1.27 1.27)) (justify left))
     )
-    (property "Footprint" "Capacitor_THT:CP_Radial_D16.0mm_P7.50mm" (at 155.9052 124.46 0)
+    (property "Footprint" "Capacitor_THT:CP_Radial_D18.0mm_P7.50mm" (at 155.9052 124.46 0)
       (effects (font (size 1.27 1.27)) hide)
     )
@@
       (effects (font (size 1.27 1.27)) (justify left))
     )
-    (property "Footprint" "Capacitor_THT:CP_Radial_D16.0mm_P7.50mm" (at 155.9052 144.78 0)
-      (effects (font (size 1.27 1.27)) hide)
-    )
+    (property "Footprint" "Capacitor_THT:CP_Radial_D18.0mm_P7.50mm" (at 155.9052 144.78 0)
+      (effects (font (size 1.27 1.27)) hide)
+    )

Commit message: Add files via upload
Parts:
- removed D10, D3, D4, D5, D6, D7, D8, D9: 1N4001, Diode_THT:D_DO-41_SOD81_P10.16mm_Horizontal, symbol Diode:1N4001
- removed J9: center tap, Connector_Pin:Pin_D1.1mm_L8.5mm_W2.5mm_FlatFork, symbol Connector:Screw_Terminal_01x01
- added D11, D3: B40C2300-1500B, Diode_THT:Diode_Bridge_19.0x3.5x10.0mm_P5.0mm, symbol Diode_Bridge:B40C2300-1500B
Connections:
- net GND2: now also D3.1 (-)
- net at F2.2: now also D11.3 (+)
- net at J9.1 (Pin_1): now also D11.2
- net at F3.2: now also D11.1 (-)
- net at J9.1 (Pin_1): now also D3.4
- net at F1.2: now also D3.3 (+)
- net at J9.1 (Pin_1): now also D11.4
- net at J9.1 (Pin_1): now also D3.2
Other:
- moved on the sheet: J9

Commit message: Add files via upload
Parts:
- removed J9 (x2): Screw_Terminal_01x01, Connector_Pin:Pin_D1.1mm_L8.5mm_W2.5mm_FlatFork, symbol Connector:Screw_Terminal_01x01
- added R11: R, Resistor_THT:R_Axial_DIN0617_L17.0mm_D6.0mm_P25.40mm_Horizontal, symbol Device:R
Connections:
- net at C10.1, F1.1, J9.1 (Pin_1)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: now also R11.1
- net at C1.1, J9.1 (Pin_1): now also R11.2
Other:
- moved on the sheet: C1, J9
